File: HydroSafeBattery.sch (EAGLE design)
At the start: 152 parts, among them P10 18650_BAT_TRAY_SMD_NON_POLAR, P11 18650_BAT_TRAY_SMD_NON_POLAR, P12 18650_BAT_TRAY_SMD_NON_POLAR, P13 18650_BAT_TRAY_SMD_NON_POLAR, P14 18650_BAT_TRAY_SMD_NON_POLAR, P15 BQ78350-R1, P2 1054500101, P3 18650_BAT_TRAY_SMD_NON_POLAR, P4 18650_BAT_TRAY_SMD_NON_POLAR, P5 18650_BAT_TRAY_SMD_NON_POLAR, P6 18650_BAT_TRAY_SMD_NON_POLAR, P7 18650_BAT_TRAY_SMD_NON_POLAR, P8 18650_BAT_TRAY_SMD_NON_POLAR, P9 18650_BAT_TRAY_SMD_NON_POLAR, Q1 BSS138, Q2 PSMN7R0-100BS, Q3 PSMN7R0-100BS, Q4 30V, 2.5A, U1 bq7694002DBT, U11 MCP2221-I/ST, U2 DMP2240, U3 DMP2240, U4 DMP2240, U5 DMP2240, U6 DMP2240, U7 DMP2240, U8 DMP2240, U9 DMP2240

Commit message: Update 2
Updates to board
Parts:
- added C3, C5: 0.1uF, SparkFun-Capacitors:0.1UF-0603-100V-10%
- added D12, D17, D22, D24, D25: GREEN, SparkFun-LED:LED-GREEN1206
- added D26: GF1, diode:GF1
- added IC1: TUSB320IRWBR, TUSB320IRWBR:TUSB320IRWBR
- added R11, R16: 1M, SparkFun-Resistors:1MOHM-0603-1/4W-5%
- added R23: 10k, SparkFun-Resistors:10KOHM-0603-1/10W-1%
- added U10: MMBTA92-7-F, MMBTA92-7-F:MMBTA92-7-F
Connections:
- new net N$22: D24.C, P15.LED4
- new net N$24: D22.C, P15.LED3
- new net N$29: D17.C, P15.LED2
- new net N$31: D12.C, P15.LED1
- new net N$36: D12.A, D17.A, D22.A, D24.A, D25.A
- new net N$38: P15.SMBC
- new net N$39: P15.SMBD
- new net N$40: P15.ALERT
- new net N$41: C5.1, P15.RBI
- new net N$45: P15.SDA
- new net N$48: P15.SCL
- new net N$49: P15.BAT
- new net N$53: P15.KEYIN
- new net N$54: P15.MRST
- new net N$55: R11.1, R16.1
- new net N$56: P15.PRECHG, R23.2
- new net N$59: R23.1, U10.B
- new net N$60: C3.1, P15.VCC, U10.E
- net GND: now also C3.2, C5.2, P15.GPIO_B, P2.GND, U11.VSS
- net N$19: now also D25.C, P15.LED5; no longer P2.GND, U11.VSS
Other:
- moved on the sheet: P2
