File: HydroSafeBattery/HydroSafeBattery.sch (EAGLE design)
At the start: 152 parts, among them P10 18650_BAT_TRAY_SMD_NON_POLAR, P11 18650_BAT_TRAY_SMD_NON_POLAR, P12 18650_BAT_TRAY_SMD_NON_POLAR, P13 18650_BAT_TRAY_SMD_NON_POLAR, P14 18650_BAT_TRAY_SMD_NON_POLAR, P15 BQ78350-R1, P2 1054500101, P3 18650_BAT_TRAY_SMD_NON_POLAR, P4 18650_BAT_TRAY_SMD_NON_POLAR, P5 18650_BAT_TRAY_SMD_NON_POLAR, P6 18650_BAT_TRAY_SMD_NON_POLAR, P7 18650_BAT_TRAY_SMD_NON_POLAR, P8 18650_BAT_TRAY_SMD_NON_POLAR, P9 18650_BAT_TRAY_SMD_NON_POLAR, Q1 BSS138, Q2 PSMN7R0-100BS, Q3 PSMN7R0-100BS, Q4 30V, 2.5A, U1 bq7694002DBT, U11 MCP2221-I/ST, U2 DMP2240, U3 DMP2240, U4 DMP2240, U5 DMP2240, U6 DMP2240, U7 DMP2240, U8 DMP2240, U9 DMP2240

Commit message: Update 2
Updates to board
Parts:
- added P1, P16, P17, P18, P19, P20, P21, P22, P23, P24, P25, P26, P27, P28, P29, P30, P31, P32, P33, P34, P35, P36, P37, P38, P39, P40, P41, P42, P43, P44, P45, P46, P47, P48, P49, P50, P51, P52, P53, P54, P55, P56, P57, P58, P59, P60, P61, P62, P63, P64, P65, P66, P67, P68, P69, P70, P71, P72, P73, P74: 18650_BAT_TRAY_SMD_NON_POLAR, Hydronalix:18650_BAT_TRAY_SMD_NON_POLAR
Connections:
- new net CELL12: P13.V-, P14.V+
- new net CELL13: P3.V-, P4.V+
- new net CELL14: P4.V-, P5.V+
- new net CELL15: P5.V-, P6.V+
- new net CELL16: P6.V-, P7.V+
- new net CELL17: P7.V-, P8.V+
- new net CELL18: P8.V-, P9.V+
- new net CELL19: P10.V+, P9.V-
- new net CELL20: P10.V-, P11.V+
- new net CELL21: P11.V-, P12.V+
- new net CELL22: P12.V-, P13.V+
- new net CELL23: P37.V-, P38.V+
- new net CELL24: P27.V-, P28.V+
- new net CELL25: P28.V-, P29.V+
- new net CELL26: P29.V-, P30.V+
- new net CELL27: P30.V-, P31.V+
- new net CELL28: P31.V-, P32.V+
- new net CELL29: P32.V-, P33.V+
- new net CELL30: P33.V-, P34.V+
- new net CELL31: P34.V-, P35.V+
- new net CELL32: P35.V-, P36.V+
- new net CELL33: P36.V-, P37.V+
- new net CELL34: P49.V-, P50.V+
- new net CELL35: P39.V-, P40.V+
- new net CELL36: P40.V-, P41.V+
- new net CELL37: P41.V-, P42.V+
- new net CELL38: P42.V-, P43.V+
- new net CELL39: P43.V-, P44.V+
- new net CELL40: P44.V-, P45.V+
- new net CELL41: P45.V-, P46.V+
- new net CELL42: P46.V-, P47.V+
- new net CELL43: P47.V-, P48.V+
- new net CELL44: P48.V-, P49.V+
- new net CELL45: P61.V-, P62.V+
- new net CELL46: P51.V-, P52.V+
- new net CELL47: P52.V-, P53.V+
- new net CELL48: P53.V-, P54.V+
- new net CELL49: P54.V-, P55.V+
- new net CELL50: P55.V-, P56.V+
- new net CELL51: P56.V-, P57.V+
- new net CELL52: P57.V-, P58.V+
- new net CELL53: P58.V-, P59.V+
- new net CELL54: P59.V-, P60.V+
- new net CELL55: P60.V-, P61.V+
- new net CELL56: P73.V-, P74.V+
- new net CELL57: P63.V-, P64.V+
- new net CELL58: P64.V-, P65.V+
- new net CELL59: P65.V-, P66.V+
- new net CELL60: P66.V-, P67.V+
- new net CELL61: P67.V-, P68.V+
- new net CELL62: P68.V-, P69.V+
- new net CELL63: P69.V-, P70.V+
- new net CELL64: P70.V-, P71.V+
- new net CELL65: P71.V-, P72.V+
- new net CELL66: P72.V-, P73.V+
- new net PACK+1: P3.V+
- new net PACK+2: P27.V+
- new net PACK+3: P39.V+
- new net PACK+4: P51.V+
- new net PACK+5: P63.V+
- net CELL1: now also P25.V-, P26.V+
- net CELL10: now also P16.V-, P17.V+
- net CELL11: now also P1.V-, P16.V+
- net CELL2: now also P24.V-, P25.V+
- net CELL3: now also P23.V-, P24.V+
- net CELL4: now also P22.V-, P23.V+
- net CELL5: now also P21.V-, P22.V+
- net CELL6: now also P20.V-, P21.V+
- net CELL7: now also P19.V-, P20.V+
- net CELL8: now also P18.V-, P19.V+
- net CELL9: now also P17.V-, P18.V+
- net GND: now also P14.V-, P26.V-, P38.V-, P50.V-, P62.V-, P74.V-
- net PACK+: now also P1.V+
